File: OpeN64/OpeN64.kicad_sch (KiCad schematic)
At the start: 270 parts, among them P6 P5, SW1 N64_SW1_Power, SW2 RESET, U13 78M05, x1 Crystal_Small, x2 Crystal_Small

Commit message: Start schematic rework - recreate RDRAM symbols
Parts:
- U11: symbol OpeN64:N64_U11_RAM_Bottom -> OpeN64:N64_U14_RAM_Top
Connections:
- net at U11.26 (IC): now also U11.6 (IC)
- net at U14.26 (IC): now also U14.6 (IC)
- net at P1.1 (NC): now also P1.35 (NC)
- no-connect marks 19 -> 13
Other:
- note added: "RDRAM A"
- note added: "RDRAM B"
- note added: "RDRAM EXP"
- moved on the sheet: C102, C103, C111, C117, C118, C119, C133, C37, C41, C42, C43, C44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

Commit message: fix reset switch symbol + footprint to correct DRC error
Connections:
- net GND: now also SW2.2 (B); no longer SW2.4 (B)
- net RSWIN: no longer SW2.2 (A)
Changed lines of the file:
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@@
 		(pin "1"
-		)
-		(pin "4"
 		)
 		(pin "2"

Commit message: update schematic symbols to conform more closely to KiCad standards
Parts:
- U9: footprint OpeN64:OpeN64_U9_RCP-NUS -> OpeN64:N64 RCP
Connections:
- net CCTLPGM is gone; now on net NMI: R24.2, U9.159 (CCTLPGM)
- net +3.3V: no longer U9.1 (VDD), U9.101 (VDD), U9.106 (VDD), U9.110 (VDD), U9.114 (VDD), U9.120 (VDD), U9.126 (VDD), U9.13 (VDD), U9.17 (VDD), U9.22 (VDD), U9.27 (VDD), U9.29 (VDD), U9.37 (VDD), U9.43 (VDD), U9.49 (VDD), U9.56 (VDD), U9.64 (VDD), U9.71 (VDD), U9.77 (VDD), U9.83 (VDD), U9.88 (VDD), U9.9 (VDD), U9.90 (VDD), U9.98 (VDD)
- net CLDRES: no longer U10.110 (ColdReset)
- net GND: no longer U9.100 (VSS), U9.105 (VSS), U9.109 (VSS), U9.113 (VSS), U9.119 (VSS), U9.12 (VSS), U9.125 (VSS), U9.16 (VSS), U9.160 (VSS), U9.2 (VSS), U9.21 (VSS), U9.28 (VSS), U9.30 (VSS), U9.36 (VSS), U9.42 (VSS), U9.48 (VSS), U9.55 (VSS), U9.63 (VSS), U9.70 (VSS), U9.76 (VSS), U9.8 (VSS), U9.82 (VSS), U9.89 (VSS), U9.91 (VSS), U9.97 (VSS)
- new net: U9.1 (VDD), U9.101 (VDD), U9.106 (VDD), U9.110 (VDD), U9.114 (VDD), U9.120 (VDD), U9.126 (VDD), U9.13 (VDD), U9.17 (VDD), U9.22 (VDD), U9.27 (VDD), U9.29 (VDD), U9.37 (VDD), U9.43 (VDD), U9.49 (VDD), U9.56 (VDD), U9.64 (VDD), U9.71 (VDD), U9.77 (VDD), U9.83 (VDD), U9.88 (VDD), U9.9 (VDD), U9.90 (VDD), U9.98 (VDD)
- new net: U9.100 (VSS), U9.105 (VSS), U9.109 (VSS), U9.113 (VSS), U9.119 (VSS), U9.12 (VSS), U9.125 (VSS), U9.16 (VSS), U9.160 (VSS), U9.2 (VSS), U9.21 (VSS), U9.28 (VSS), U9.30 (VSS), U9.36 (VSS), U9.42 (VSS), U9.48 (VSS), U9.55 (VSS), U9.63 (VSS), U9.70 (VSS), U9.76 (VSS), U9.8 (VSS), U9.82 (VSS), U9.89 (VSS), U9.91 (VSS), U9.97 (VSS)
- new net CLD_RST: U10.110 (ColdReset)
Other:
- moved on the sheet: C131, C132, C134, C5, C6, C7, C70, C75, C76, C77, C78, C8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
